File: EncoderBoard.kicad_pcb (KiCad board)
At the start: 2 copper layers, 28.8 x 27.8 mm, 12 parts, among them J1 Conn_01x06_MountingPin, J2 Conn_01x05_MountingPin, J3 Conn_01x05_MountingPin, J4 Conn_01x03_MountingPin, U1 AS5047P

Commit message: Update for V2
Parts:
- added R1: 10k, Resistor_SMD:R_0402_1005Metric, F.Cu at (150.4, 95.7)
- added R2: 10k, Resistor_SMD:R_0402_1005Metric, F.Cu at (146.8, 95.2)
- added R3: 10k, Resistor_SMD:R_0402_1005Metric, F.Cu at (144.7, 100.6)
- C1, C2: footprint Capacitor_SMD:C_0603_1608Metric -> Capacitor_SMD:C_0402_1005Metric
- moved C2 4.45 mm to (153.4, 96.0), turned to 90 degrees
- moved C1 0.22 mm to (156.8, 97.3)
Routing:
- net VDD: track 45.4 -> 51.3 mm
- net Net-(J1-Pin_2): track 6.79 -> 10.9 mm
- net GND: track 3.35 -> 6.43 mm, vias 2 -> 4
- net Net-(JP1-A): track 2.69 -> 5.41 mm
- net Net-(J2-Pin_3): track 13.6 -> 15.2 mm, vias 0 -> 2
- net Net-(J1-Pin_3): track 7.46 -> 8.35 mm
- net Net-(J1-Pin_5): track 8.33 -> 9.14 mm
Other:
- board text added: "V2"
