File: EncoderBoard.kicad_sch (KiCad schematic)
At the start: 12 parts, among them J1 Conn_01x06_MountingPin, J2 Conn_01x05_MountingPin, J3 Conn_01x05_MountingPin, J4 Conn_01x03_MountingPin, U1 AS5047P

Commit message: Update for V2
Parts:
- added R1, R2, R3: 10k, Resistor_SMD:R_0402_1005Metric, symbol Device:R_Small_US
- C1, C2: footprint Capacitor_SMD:C_0603_1608Metric -> Capacitor_SMD:C_0402_1005Metric
Connections:
- net GND: now also R2.1, R3.1
- net VDD: now also R1.1
- net at J1.2 (Pin_2), U1.1 (~{CS}): now also R1.2
- net at J1.3 (Pin_3), U1.2 (CLK): now also R2.2
- net at J1.5 (Pin_5), U1.4 (MOSI): now also R3.2
